File: be6502x sbc FIRST FAB/be6502x.kicad_pcb (KiCad board)
At the start: 2 copper layers, 118.4 x 109.3 mm, 44 parts, among them J0 Regulated +5v In, J1 IO Port A, J2 IO Port B, J3 Unassigned Bus Signals, J4 Control Signals, P1 BE6502X Bus, P2 BE6502X Bus, P3 BE6502X Bus, SW1 Reset, U1 W65C02SxP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

Commit message: Add files via upload
Parts:
- D2: value CA1 LED -> CA2 LED
Other:
- board text added: "CA2"
- board text removed: "CA1"
Changed lines of the file:
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@@
     (add_net "Net-(JP1-Pad2)")
     (add_net "Net-(JP3-Pad2)")
+    (add_net "Net-(U1-Pad3)")
+    (add_net "Net-(U1-Pad35)")
+    (add_net "Net-(U1-Pad39)")
+    (add_net "Net-(U3-Pad11)")
     (add_net PA0)
     (add_net PA1)
@@
       (effects (font (size 1 1) (thickness 0.15)))
     )
-    (fp_text value "CA1 LED" (at 1.27 3.46 90) (layer F.Fab)
+    (fp_text value "CA2 LED" (at 1.27 3.46 90) (layer F.Fab)
       (effects (font (size 1 1) (thickness 0.15)))
     )
@@
     (effects (font (size 1.2 1.2) (thickness 0.1524)))
   )
-  (gr_text CA1 (at 98.1075 137.668 90) (layer F.SilkS)
+  (gr_text CA2 (at 98.1075 137.668 90) (layer F.SilkS)
     (effects (font (size 1.2 1.2) (thickness 0.1524)))
   )
