File: be6502x sbc FIRST FAB/be6502x.sch (KiCad schematic (older format))
At the start: 44 parts, among them J0 Regulated +5v In, J1 IO Port A, J2 IO Port B, J3 Unassigned Bus Signals, J4 Control Signals, P1 BE6502X Bus, P2 BE6502X Bus, P3 BE6502X Bus, SW1 Reset, U1 W65C02SxP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

Commit message: Add files via upload
Parts:
- D2: value CA1 LED -> CA2 LED
Changed lines of the file:
@@
 P 1500 4700
 F 0 "D2" H 1493 4917 50  0000 C CNN
-F 1 "CA1 LED" H 1493 4826 50  0000 C CNN
+F 1 "CA2 LED" H 1493 4826 50  0000 C CNN
 F 2 "LED_THT:LED_D4.0mm" H 1500 4700 50  0001 C CNN
 F 3 "~" H 1500 4700 50  0001 C CNN
@@
 Connection ~ 4450 6050
 Connection ~ 750  5050
-Wire Bus Line
-	2600 4800 2600 5750
-Wire Bus Line
-	6900 1400 6900 2850
-Wire Bus Line
-	3050 3250 3050 3950
-Wire Bus Line
-	4750 1600 4750 3950
-Wire Bus Line
-	3100 1550 3100 3050
-Wire Bus Line
-	3550 1550 3550 3100
-Wire Bus Line
-	5350 1400 5350 3100
-Wire Bus Line
-	6750 1600 6750 3950
 $Comp
 L power:+5V #PWR0101
@@
 	0    1    1    0
 $EndComp
+Wire Bus Line
+	2600 4800 2600 5750
+Wire Bus Line
+	6900 1400 6900 2850
+Wire Bus Line
+	3050 3250 3050 3950
+Wire Bus Line
+	4750 1600 4750 3950
+Wire Bus Line
+	3100 1550 3100 3050
+Wire Bus Line
+	3550 1550 3550 3100
+Wire Bus Line
+	5350 1400 5350 3100
+Wire Bus Line
+	6750 1600 6750 3950
 $EndSCHEMATC
